File: 02_ECAD_ECU/STM32F446_carrier_board/_autosave-stm32f446re_carrier_board.kicad_pcb (KiCad board)
At the start: 4 copper layers, 53 x 60.6 mm, 62 parts, among them IC1 MP2303ADN-LF, J1 POWER, J2 FX10A-80P_8-SV_71_, J3 C10418, J4 SWD, Q1 AO3401A, SW1 SW_SPDT, U1 STM32F446RETx, U2 USBLC6-2SC6, U3 W25N01GVZEIG_TR, Y1 16MHz, Y2 32.768kHz

Commit message: carrierboard stm32f446 finished v0.1
Other:
- board text added: "Tellur - STM32F446 V0.1 by Max Altrichter"
- board text removed: "Carrierboard- STM32F446 V0.1 by Max Altrichter"
