File: 02_ECAD_ECU/twoLevelInverter/twoLevelInverter/step_down_converter_3V3.kicad_sch (KiCad schematic)
At the start: 17 parts, among them U1 290mA, U10 30k, U11 2.4k, U12 22u, U13 15u, U14 RED, U15 1k, U2 100k, U3 68k, U4 MP2303ADN-LF, U5 10nF, U6 100nF, U7 3.3nF, U8 5.6k, U9 10k

Commit message: V1.0  not reviewed
Parts:
- removed C17: 10uF/24V, Capacitor_SMD:C_1206_3216Metric, symbol Device:C_Polarized_Small
- removed FB1: 600 @ 600MHz, Inductor_SMD:L_1206_3216Metric, symbol Device:FerriteBead_Small
- removed U1: 290mA, Fuse:Fuse_1206_3216Metric, symbol Device:Polyfuse_Small
- removed U10: 30k, Resistor_SMD:R_0805_2012Metric, symbol Device:R_Small
- removed U11: 2.4k, Resistor_SMD:R_0603_1608Metric, symbol Device:R_Small
- removed U12: 22u, Capacitor_SMD:C_0805_2012Metric, symbol Device:C_Small
- removed U13: 15u, max_KiCAD_lib:LVS505020-150M-N, symbol Device:L_Small
- removed U2: 100k, Resistor_SMD:R_1206_3216Metric, symbol Device:R_Small
- removed U3: 68k, Resistor_SMD:R_0805_2012Metric, symbol Device:R_Small
- removed U4: MP2303ADN-LF, max_KiCAD_lib:SOIC127P600X170-9N, symbol max_KiCAD_lib:MP2303ADN-LF
- removed U5: 10nF, Capacitor_SMD:C_0805_2012Metric, symbol Device:C_Small
- removed U6: 100nF, Capacitor_SMD:C_0603_1608Metric, symbol Device:C_Small
- removed U7: 3.3nF, Capacitor_SMD:C_0603_1608Metric, symbol Device:C_Small
- removed U8: 5.6k, Resistor_SMD:R_0603_1608Metric, symbol Device:R_Small
- removed U9: 10k, Resistor_SMD:R_1206_3216Metric, symbol Device:R_Small
- added C17: 10 nF, Capacitor_SMD:C_1206_3216Metric, symbol Device:C_Small
- added C18: 100uF, max_KiCAD_lib:100uF_wuerth, symbol Device:C_Polarized
- added C19: 68 uF, max_KiCAD_lib:68uFcap, symbol Device:C_Polarized
- added D3: D_Schottky, max_KiCAD_lib:schottydiode50V, symbol Device:D_Schottky
- added IC8: LM2675N-3.3_NOPB, max_KiCAD_lib:LM2675N, symbol CustomLib:LM2675N-3.3_NOPB
- added L2: 47uH, Capacitor_SMD:C_0805_2012Metric, symbol Device:L_Small
- U14: value RED -> 3V3; footprint LED_SMD:LED_0603_1608Metric -> LED_SMD:LED_1206_3216Metric
Connections:
- net 3V3: now also C19.1, IC8.4 (FB), L2.2
- net GND: now also C18.2, C19.2, D3.2 (A), IC8.6 (GND)
- net VCC: now also C18.1, IC8.7 (VIN)
- new net: C17.1, D3.1 (K), IC8.8 (VSW), L2.1
- new net: C17.2, IC8.1 (CB)
- no-connect marks 1 -> 3
Other:
- note removed: "6.3V CERAMICx2"
- moved on the sheet: U14, U15

Commit message: orderd, added gerber files
Parts:
- U14: footprint LED_SMD:LED_1206_3216Metric -> LED_SMD:LED_0805_2012Metric
Changed lines of the file:
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@@
       (effects (font (size 1.27 1.27)) (justify right))
     )
-    (property "Footprint" "LED_SMD:LED_1206_3216Metric" (id 2) (at 223.52 91.44 90)
+    (property "Footprint" "LED_SMD:LED_0805_2012Metric" (id 2) (at 223.52 91.44 90)
       (effects (font (size 1.27 1.27)) hide)
     )
