File: 02_ECAD_ECU/twoLevelInverter/twoLevelInverter/step_down_converter_5V.kicad_sch (KiCad schematic)
At the start: 11 parts, among them IC1 MP9486AGN-Z

Commit message: V1.0  not reviewed
Parts:
- added U1: 5V, LED_SMD:LED_1206_3216Metric, symbol Device:LED_Small
- added U2: 1k, Resistor_SMD:R_1206_3216Metric, symbol Device:R_Small
Connections:
- net En is gone; now on net EN: IC1.6 (DIM), IC1.7 (EN)
- net GND: now also IC1.9 (EP), U2.2
- net V_out: now also U1.2 (A)
- new net: U1.1 (K), U2.1
Changed lines of the file:
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@@
   (junction (at 224.79 85.09) (diameter 0) (color 0 0 0 0)
   )
+  (junction (at 243.84 85.09) (diameter 0) (color 0 0 0 0)
+  )
   (junction (at 97.79 83.82) (diameter 0) (color 0 0 0 0)
   )
@@
   (junction (at 110.49 83.82) (diameter 0) (color 0 0 0 0)
   )
+  (junction (at 147.32 105.41) (diameter 0) (color 0 0 0 0)
+  )
   (junction (at 198.12 85.09) (diameter 0) (color 0 0 0 0)
   )
@@
   )
   (no_connect (at 132.08 97.79))
-  (wire (pts (xy 224.79 85.09) (xy 234.95 85.09))
-    (stroke (width 0) (type default) (color 0 0 0 0))
-  )
   (wire (pts (xy 21.59 21.59) (xy 29.21 21.59))
     (stroke (width 0) (type default) (color 0 0 0 0))
@@
     (stroke (width 0) (type default) (color 0 0 0 0))
   )
+  (wire (pts (xy 243.84 99.06) (xy 243.84 101.6))
+    (stroke (width 0) (type default) (color 0 0 0 0))
+  )
   (wire (pts (xy 184.15 85.09) (xy 198.12 85.09))
     (stroke (width 0) (type default) (color 0 0 0 0))
@@
     (stroke (width 0) (type default) (color 0 0 0 0))
   )
-  (wire (pts (xy 147.32 104.14) (xy 147.32 109.22))
+  (wire (pts (xy 147.32 104.14) (xy 147.32 105.41))
+    (stroke (width 0) (type default) (color 0 0 0 0))
+  )
+  (wire (pts (xy 224.79 85.09) (xy 243.84 85.09))
     (stroke (width 0) (type default) (color 0 0 0 0))
   )
@@
     (stroke (width 0) (type default) (color 0 0 0 0))
   )
+  (wire (pts (xy 243.84 92.71) (xy 243.84 93.98))
+    (stroke (width 0) (type default) (color 0 0 0 0))
+  )
   (wire (pts (xy 127 95.25) (xy 132.08 95.25))
     (stroke (width 0) (type default) (color 0 0 0 0))
@@
     (stroke (width 0) (type default) (color 0 0 0 0))
   )
+  (wire (pts (xy 144.78 104.14) (xy 144.78 105.41))
+    (stroke (width 0) (type default) (color 0 0 0 0))
+  )
   (wire (pts (xy 162.56 71.12) (xy 162.56 85.09))
     (stroke (width 0) (type default) (color 0 0 0 0))
@@
     (stroke (width 0) (type default) (color 0 0 0 0))
   )
+  (wire (pts (xy 144.78 105.41) (xy 147.32 105.41))
+    (stroke (width 0) (type default) (color 0 0 0 0))
+  )
   (wire (pts (xy 184.15 97.79) (xy 184.15 101.6))
     (stroke (width 0) (type default) (color 0 0 0 0))
@@
     (stroke (width 0) (type default) (color 0 0 0 0))
   )
+  (wire (pts (xy 147.32 105.41) (xy 147.32 109.22))
+    (stroke (width 0) (type default) (color 0 0 0 0))
+  )
+  (wire (pts (xy 243.84 85.09) (xy 243.84 87.63))
+    (stroke (width 0) (type default) (color 0 0 0 0))
+  )
   (wire (pts (xy 110.49 83.82) (xy 132.08 83.82))
+    (stroke (width 0) (type default) (color 0 0 0 0))
+  )
+  (wire (pts (xy 243.84 85.09) (xy 247.65 85.09))
     (stroke (width 0) (type default) (color 0 0 0 0))
   )
@@
     (effects (font (size 1.27 1.27)) (justify left bottom))
   )
-  (label "EN" (at 29.21 21.59 0)
+  (label "EN_5V" (at 29.21 21.59 0)
     (effects (font (size 1.27 1.27)) (justify left bottom))
   )
@@
     (effects (font (size 1.27 1.27)) (justify left bottom))
   )
-  (label "V_out" (at 234.95 85.09 0)
-    (effects (font (size 1.27 1.27)) (justify left bottom))
-  )
-  (label "En" (at 88.9 95.25 180)
+  (label "V_out" (at 247.65 85.09 0)
+    (effects (font (size 1.27 1.27)) (justify left bottom))
+  )
+  (label "EN_5V" (at 88.9 95.25 180)
     (effects (font (size 1.27 1.27)) (justify right bottom))
   )
   (label "V_in" (at 29.21 19.05 0)
+    (effects (font (size 1.27 1.27)) (justify left bottom))
+  )
+  (label "GND" (at 243.84 101.6 0)
     (effects (font (size 1.27 1.27)) (justify left bottom))
   )
@@
     )
     (property "Datasheet" "~" (id 3) (at 184.15 104.14 0)
+      (effects (font (size 1.27 1.27)) hide)
+    )
+    (pin "1")
+    (pin "2")
+  )
+  (symbol (lib_id "Device:R_Small") (at 243.84 96.52 0) (mirror y) (unit 1)
+    (in_bom yes) (on_board yes)
+    (property "Reference" "U2" (id 0) (at 246.38 95.25 0))
+    (property "Value" "1k" (id 1) (at 247.65 97.79 0))
+    (property "Footprint" "Resistor_SMD:R_1206_3216Metric" (id 2) (at 243.84 96.52 0)
+      (effects (font (size 1.27 1.27)) hide)
+    )
+    (property "Datasheet" "~" (id 3) (at 243.84 96.52 0)
+      (effects (font (size 1.27 1.27)) hide)
+    )
+    (property "LCSC part #" "C4410" (id 4) (at 243.84 96.52 0)
       (effects (font (size 1.27 1.27)) hide)
     )
@@
       (effects (font (size 1.27 1.27)) hide)
     )
+    (pin "1")
+    (pin "2")
+  )
+  (symbol (lib_id "Device:LED_Small") (at 243.84 90.17 90) (unit 1)
+    (in_bom yes) (on_board yes)
+    (property "Reference" "U1" (id 0) (at 245.618 89.0016 90)
+      (effects (font (size 1.27 1.27)) (justify right))
+    )
+    (property "Value" "5V" (id 1) (at 245.618 91.313 90)
+      (effects (font (size 1.27 1.27)) (justify right))
+    )
+    (property "Footprint" "LED_SMD:LED_1206_3216Metric" (id 2) (at 243.84 90.17 90)
+      (effects (font (size 1.27 1.27)) hide)
+    )
+    (property "Datasheet" "~" (id 3) (at 243.84 90.17 90)
+      (effects (font (size 1.27 1.27)) hide)
+    )
+    (property "LCSC part #" "C2286" (id 4) (at 243.84 90.17 0)
+      (effects (font (size 1.27 1.27)) hide)
+    )

Commit message: orderd, added gerber files
Parts:
- U1: footprint LED_SMD:LED_1206_3216Metric -> LED_SMD:LED_0805_2012Metric
Changed lines of the file:
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@@
       (effects (font (size 1.27 1.27)) (justify right))
     )
-    (property "Footprint" "LED_SMD:LED_1206_3216Metric" (id 2) (at 243.84 90.17 90)
+    (property "Footprint" "LED_SMD:LED_0805_2012Metric" (id 2) (at 243.84 90.17 90)
       (effects (font (size 1.27 1.27)) hide)
     )
